File: circuits/SimpleClock/SimpleClock/SimpleClock.kicad_sch (KiCad schematic)
At the start: 31 parts, among them J1 Screw_Terminal_01x02, J2 AVR-ISP-6, SW1 SW_SPDT, SW2 SW_Push, SW3 SW_Push, SW4 SW_Push, SW5 SW_Push, U1 ATtiny2313-20P, U2 KW4-56NCWB-P-Y

Commit message: Fix schematics and coding
Connections:
- net at U2.10 (Di3): now also U1.13 (PB1); no longer U1.14 (PB2)
- net at U2.11 (Di2): now also U1.14 (PB2); no longer U1.13 (PB1)
- net at U2.14 (Di1): now also U1.15 (PB3); no longer U1.12 (PB0)
- net at U2.6 (Di4): now also U1.12 (PB0); no longer U1.15 (PB3)
Changed lines of the file:
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@@
     (rev "1")
     (company "Out-of-Band Development")
+    (comment 1 "Designer: Matthew Whited")
   )
   (junction (at 36.83 93.98) (diameter 0) (color 0 0 0 0)
@@
     (stroke (width 0) (type default) (color 0 0 0 0))
   )
-  (wire (pts (xy 248.92 29.21) (xy 248.92 134.62))
+  (wire (pts (xy 248.92 29.21) (xy 248.92 119.38))
     (stroke (width 0) (type default) (color 0 0 0 0))
   )
@@
     (stroke (width 0) (type default) (color 0 0 0 0))
   )
+  (wire (pts (xy 250.19 124.46) (xy 250.19 27.94))
+    (stroke (width 0) (type default) (color 0 0 0 0))
+  )
   (wire (pts (xy 45.72 88.9) (xy 36.83 88.9))
     (stroke (width 0) (type default) (color 0 0 0 0))
@@
     (stroke (width 0) (type default) (color 0 0 0 0))
   )
-  (wire (pts (xy 238.76 119.38) (xy 252.73 119.38))
+  (wire (pts (xy 238.76 129.54) (xy 251.46 129.54))
     (stroke (width 0) (type default) (color 0 0 0 0))
   )
@@
     (stroke (width 0) (type default) (color 0 0 0 0))
   )
-  (wire (pts (xy 250.19 129.54) (xy 250.19 27.94))
-    (stroke (width 0) (type default) (color 0 0 0 0))
-  )
   (wire (pts (xy 149.86 67.31) (xy 149.86 26.67))
     (stroke (width 0) (type default) (color 0 0 0 0))
@@
     (stroke (width 0) (type default) (color 0 0 0 0))
   )
-  (wire (pts (xy 251.46 26.67) (xy 251.46 124.46))
+  (wire (pts (xy 251.46 26.67) (xy 251.46 129.54))
     (stroke (width 0) (type default) (color 0 0 0 0))
   )
@@
     (stroke (width 0) (type default) (color 0 0 0 0))
   )
+  (wire (pts (xy 238.76 134.62) (xy 252.73 134.62))
+    (stroke (width 0) (type default) (color 0 0 0 0))
+  )
   (wire (pts (xy 181.61 73.66) (xy 182.88 73.66))
     (stroke (width 0) (type default) (color 0 0 0 0))
@@
     (stroke (width 0) (type default) (color 0 0 0 0))
   )
-  (wire (pts (xy 251.46 124.46) (xy 238.76 124.46))
-    (stroke (width 0) (type default) (color 0 0 0 0))
-  )
   (wire (pts (xy 144.78 80.01) (xy 162.56 80.01))
     (stroke (width 0) (type default) (color 0 0 0 0))
@@
     (stroke (width 0) (type default) (color 0 0 0 0))
   )
-  (wire (pts (xy 238.76 134.62) (xy 248.92 134.62))
-    (stroke (width 0) (type default) (color 0 0 0 0))
-  )
   (wire (pts (xy 210.82 55.88) (xy 210.82 64.77))
     (stroke (width 0) (type default) (color 0 0 0 0))
@@
     (stroke (width 0) (type default) (color 0 0 0 0))
   )
+  (wire (pts (xy 238.76 124.46) (xy 250.19 124.46))
+    (stroke (width 0) (type default) (color 0 0 0 0))
+  )
   (wire (pts (xy 67.31 68.58) (xy 50.8 68.58))
     (stroke (width 0) (type default) (color 0 0 0 0))
@@
     (stroke (width 0) (type default) (color 0 0 0 0))
   )
-  (wire (pts (xy 252.73 119.38) (xy 252.73 25.4))
+  (wire (pts (xy 252.73 25.4) (xy 252.73 134.62))
     (stroke (width 0) (type default) (color 0 0 0 0))
   )
@@
     (stroke (width 0) (type default) (color 0 0 0 0))
   )
-  (wire (pts (xy 238.76 129.54) (xy 250.19 129.54))
-    (stroke (width 0) (type default) (color 0 0 0 0))
-  )
   (wire (pts (xy 137.16 97.79) (xy 157.48 97.79))
     (stroke (width 0) (type default) (color 0 0 0 0))
@@
     (stroke (width 0) (type default) (color 0 0 0 0))
   )
+  (wire (pts (xy 238.76 119.38) (xy 248.92 119.38))
+    (stroke (width 0) (type default) (color 0 0 0 0))
+  )
