File: circuits/DiodeLogicBoards/PROM/MemoryByte.kicad_sch (KiCad schematic)
At the start: 0 parts

Commit message: update circuits
Parts:
- added D1, D2, D3, D4, D5, D6, D7, D8: 1N4148, Diode_THT:D_DO-35_SOD27_P7.62mm_Horizontal, symbol Diode:1N4148
- added SW1: SW_DIP_x08, Package_DIP:DIP-16_W7.62mm, symbol Switch:SW_DIP_x08
Connections:
- new net: D8.1 (K), SW1.8
- new net: D4.1 (K), SW1.4
- new net: D3.1 (K), SW1.3
- new net: D1.1 (K), SW1.1
- new net: D2.1 (K), SW1.2
- new net: D6.1 (K), SW1.6
- new net: D5.1 (K), SW1.5
- new net: D7.1 (K), SW1.7
- new net ByteSelect: SW1.10, SW1.11, SW1.12, SW1.13, SW1.14, SW1.15, SW1.16, SW1.9
- new net Data0: D1.2 (A)
- new net Data1: D2.2 (A)
- new net Data2: D3.2 (A)
- new net Data3: D4.2 (A)
- new net Data4: D5.2 (A)
- new net Data5: D6.2 (A)
- new net Data6: D7.2 (A)
- new net Data7: D8.2 (A)
Other:
- company: (none) -> Out-of-Band Development
- title: (none) -> Diode Logic DIP PROM
