File: circuits/DiodeLogicBoards/PROM/PROM.kicad_sch (KiCad schematic)
At the start: 0 parts

Commit message: update circuits
Parts:
- added J1: Conn_01x28_Pin, symbol Connector:Conn_01x28_Pin
Connections:
- new net Byte 0: J1.17 (Pin_17)
- new net Byte 1: J1.16 (Pin_16)
- new net Byte 2: J1.15 (Pin_15)
- new net Byte 3: J1.14 (Pin_14)
- new net Byte 4: J1.13 (Pin_13)
- new net Byte 5: J1.12 (Pin_12)
- new net Byte 6: J1.11 (Pin_11)
- new net Byte 7: J1.10 (Pin_10)
- new net Byte 8: J1.9 (Pin_9)
- new net Byte 9: J1.8 (Pin_8)
- new net Byte A: J1.7 (Pin_7)
- new net Byte B: J1.6 (Pin_6)
- new net Byte C: J1.5 (Pin_5)
- new net Byte D: J1.4 (Pin_4)
- new net Byte E: J1.3 (Pin_3)
- new net Byte F: J1.2 (Pin_2)
- new net Data 0: J1.20 (Pin_20)
- new net Data 1: J1.21 (Pin_21)
- new net Data 2: J1.22 (Pin_22)
- new net Data 3: J1.23 (Pin_23)
- new net Data 4: J1.24 (Pin_24)
- new net Data 5: J1.25 (Pin_25)
- new net Data 6: J1.26 (Pin_26)
- new net Data 7: J1.27 (Pin_27)
- no-connect marks 0 -> 4
Other:
- sheet MemoryByte renamed MemoryByte 0
- added sheet MemoryByte 1 (MemoryByte.kicad_sch)
- added sheet MemoryByte 2 (MemoryByte.kicad_sch)
- added sheet MemoryByte 3 (MemoryByte.kicad_sch)
- added sheet MemoryByte 4 (MemoryByte.kicad_sch)
- added sheet MemoryByte 5 (MemoryByte.kicad_sch)
- added sheet MemoryByte 6 (MemoryByte.kicad_sch)
- added sheet MemoryByte 7 (MemoryByte.kicad_sch)
- added sheet MemoryByte 8 (MemoryByte.kicad_sch)
- added sheet MemoryByte 9 (MemoryByte.kicad_sch)
- added sheet MemoryByte A (MemoryByte.kicad_sch)
- added sheet MemoryByte B (MemoryByte.kicad_sch)
- added sheet MemoryByte C (MemoryByte.kicad_sch)
- added sheet MemoryByte D (MemoryByte.kicad_sch)
- added sheet MemoryByte E (MemoryByte.kicad_sch)
- added sheet MemoryByte F (MemoryByte.kicad_sch)
- sheet MemoryByte 0 ports: added ByteSelect, Data0, Data1, Data2, Data3, Data4, Data5, Data6, Data7; removed none
- company: (none) -> Out-of-Band Development
- title: (none) -> Diode Logic DIP PROM
