File: circuits/AnalogCalculator/AnalogComputer/AnalogComputer.kicad_pcb (KiCad board)
At the start: 2 copper layers, 135 x 80 mm, 85 parts, among them J1 Conn_02x14_Odd_Even, J2 Conn_02x14_Odd_Even, J3 Conn_02x14_Odd_Even, J4 Conn_01x03_Pin, U1 LM324, U2 LM324, U3 LM324, U4 LM324, U5 LM324, U6 LM324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

Commit message: update circuits
Parts:
- added J5: Conn_02x14_Odd_Even, Connector_PinHeader_2.54mm:PinHeader_2x14_P2.54mm_Vertical, F.Cu at (215.3, 69.6)
- added J6: Conn_02x14_Odd_Even, Connector_PinHeader_2.54mm:PinHeader_2x14_P2.54mm_Vertical, F.Cu at (222.5, 69.6)
Connections:
- net +12V renamed VCC
- net -12V renamed VSS

Commit message: update layount
Parts:
- added J7: Conn_02x14_Odd_Even, Connector_PinHeader_2.54mm:PinHeader_2x14_P2.54mm_Vertical, F.Cu at (108.2, 140.5)
- added R49: 1k, Resistor_THT:R_Axial_DIN0204_L3.6mm_D1.6mm_P2.54mm_Vertical, F.Cu at (174.7, 90.0)
- added R50: 1k, Resistor_THT:R_Axial_DIN0204_L3.6mm_D1.6mm_P2.54mm_Vertical, F.Cu at (174.7, 82.3)
- added R51: 1k, Resistor_THT:R_Axial_DIN0204_L3.6mm_D1.6mm_P2.54mm_Vertical, F.Cu at (153.7, 89.8)
- added R52: 1k, Resistor_THT:R_Axial_DIN0204_L3.6mm_D1.6mm_P2.54mm_Vertical, F.Cu at (153.7, 81.8)
- added R53: 10k, Resistor_THT:R_Axial_DIN0204_L3.6mm_D1.6mm_P2.54mm_Vertical, F.Cu at (155.7, 109.5)
- added R54: 10k, Resistor_THT:R_Axial_DIN0204_L3.6mm_D1.6mm_P2.54mm_Vertical, F.Cu at (155.3, 125.5)
- added R55: 10k, Resistor_THT:R_Axial_DIN0204_L3.6mm_D1.6mm_P2.54mm_Vertical, F.Cu at (168.0, 132.0)
- added R56: 10k, Resistor_THT:R_Axial_DIN0204_L3.6mm_D1.6mm_P2.54mm_Vertical, F.Cu at (168.7, 100.5)
- added REF**: MountingHole_2.2mm_M2_Pad_TopBottom, MountingHole:MountingHole_2.2mm_M2_Pad_TopBottom, F.Cu at (145.5, 86.5)
- added REF**: MountingHole_2.2mm_M2_Pad_TopBottom, MountingHole:MountingHole_2.2mm_M2_Pad_TopBottom, F.Cu at (177.0, 131.5)
- added REF**: MountingHole_2.2mm_M2_Pad_TopBottom, MountingHole:MountingHole_2.2mm_M2_Pad_TopBottom, F.Cu at (65.0, 139.5)
- added REF**: MountingHole_2.2mm_M2_Pad_TopBottom, MountingHole:MountingHole_2.2mm_M2_Pad_TopBottom, F.Cu at (65.5, 70.0)
- added RN1: 10k, Resistor_THT:R_Array_SIP5, F.Cu at (158.5, 93.3)
- added RN2: 10k, Resistor_THT:R_Array_SIP5, F.Cu at (166.4, 93.3)
- added RN3: 10k, Resistor_THT:R_Array_SIP5, F.Cu at (166.9, 78.8)
- added RN4: 10k, Resistor_THT:R_Array_SIP5, F.Cu at (158.5, 78.8)
- added RN5: 10k, Resistor_THT:R_Array_SIP5, F.Cu at (157.5, 112.5)
- added RN6: 10k, Resistor_THT:R_Array_SIP9, F.Cu at (168.0, 128.5)
- added RN7: 10k, Resistor_THT:R_Array_SIP5, F.Cu at (157.5, 122.5)
- added RN8: 10k, Resistor_THT:R_Array_SIP9, F.Cu at (168.5, 104.0)
- added U10: LM324, Package_DIP:DIP-14_W7.62mm_Socket, F.Cu at (156.4, 89.8)
- added U11: LM324, Package_DIP:DIP-14_W7.62mm_Socket, F.Cu at (160.9, 109.8)
- added U12: LM324, Package_DIP:DIP-14_W7.62mm_Socket, F.Cu at (133.2, 76.9)
- added U13: LM324, Package_DIP:DIP-14_W7.62mm_Socket, F.Cu at (133.0, 97.3)
- added U14: LM324, Package_DIP:DIP-14_W7.62mm_Socket, F.Cu at (133.5, 117.3)
- D22: moved to B.Cu
- moved J4 119.5 mm to (176.5, 116.0)
- moved J6 81.2 mm to (178.5, 138.0), turned to -90 degrees
- moved J2 79.4 mm to (70.5, 140.5)
- moved R47 71.0 mm to (111.2, 119.2), turned to 90 degrees
- moved R45 70.6 mm to (111.1, 99.7), turned to 90 degrees
- moved R37 69.6 mm to (111.1, 78.7), turned to 90 degrees
- moved J5 69.4 mm to (145.8, 71.5), turned to 90 degrees
- moved R44 64.7 mm to (111.1, 112.7), turned to 90 degrees
- moved R48 64.6 mm to (111.2, 132.7), turned to 90 degrees
- moved R39 64.3 mm to (111.1, 92.2), turned to 90 degrees
- moved R43 52.5 mm to (129.6, 112.7), turned to 90 degrees
- moved R46 52.4 mm to (129.7, 132.7), turned to 90 degrees
- moved R38 51.1 mm to (129.6, 92.2), turned to 90 degrees
- moved U9 47.3 mm to (116.7, 117.4)
- moved U7 46.8 mm to (116.5, 76.9)
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Routing:
- net GND: track 382.9 -> 0.00 mm, vias 1 -> 0
- net VSS: track 278.7 -> 0.00 mm
- net VCC: track 248.5 -> 0.00 mm, vias 2 -> 0
- net /LogOut5: track 135.6 -> 0.00 mm
- net /InvertOut9: track 98.3 -> 0.00 mm
- net /InvertOut5: track 95.7 -> 0.00 mm, vias 2 -> 0
- net /InvertOut10: track 95.0 -> 0.00 mm
- net /InvertOut11: track 88.9 -> 0.00 mm
- net /InvertOut8: track 87.7 -> 0.00 mm
- net /AlogIn6: track 87.4 -> 0.00 mm
- net /InvertIn8: track 84.0 -> 0.00 mm
- net /ALogOut6: track 79.6 -> 0.00 mm
- net /LogIn6: track 79.0 -> 0.00 mm
- net /AlogIn7: track 78.3 -> 0.00 mm
- net /LogOut6: track 77.7 -> 0.00 mm
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- added copper zone on B.Cu, net VSS
- added copper zone on F.Cu, net VSS
Other:
- board size 135 x 80 mm -> 120.7 x 80 mm
