File: circuits/AnalogCalculator/AnalogComputer/AnalogComputer.kicad_sch (KiCad schematic)
At the start: 4 parts, among them J1 Conn_02x14_Odd_Even, J2 Conn_02x14_Odd_Even, J3 Conn_02x14_Odd_Even, J4 Conn_01x03_Pin

Commit message: update circuits
Parts:
- added J5, J6: Conn_02x14_Odd_Even, Connector_PinHeader_2.54mm:PinHeader_2x14_P2.54mm_Vertical, symbol Connector_Generic:Conn_02x14_Odd_Even
Connections:
- net +12V renamed VCC
- net -12V renamed VSS
- new net In 10k A 0: J5.1 (Pin_1)
- new net In 10k A 1: J5.3 (Pin_3)
- new net In 10k A 2: J5.5 (Pin_5)
- new net In 10k A 3: J5.7 (Pin_7)
- new net In 10k B 0: J5.2 (Pin_2)
- new net In 10k B 1: J5.4 (Pin_4)
- new net In 10k B 2: J5.6 (Pin_6)
- new net In 10k B 3: J5.8 (Pin_8)
- new net In 10k C 0: J5.15 (Pin_15)
- new net In 10k C 1: J5.17 (Pin_17)
- new net In 10k C 2: J5.19 (Pin_19)
- new net In 10k C 3: J5.21 (Pin_21)
- new net In 10k D 0: J5.16 (Pin_16)
- new net In 10k D 1: J5.18 (Pin_18)
- new net In 10k D 2: J5.20 (Pin_20)
- new net In 10k D 3: J5.22 (Pin_22)
- new net In 1k A 4: J5.9 (Pin_9)
- new net In 1k B 4: J5.10 (Pin_10)
- new net In 1k C 4: J5.23 (Pin_23)
- new net In 1k D 4: J5.24 (Pin_24)
- new net In a 0: J6.1 (Pin_1)
- new net In a 1: J6.3 (Pin_3)
- new net In a 2: J6.5 (Pin_5)
- new net In a 3: J6.7 (Pin_7)
- new net In b 0: J6.2 (Pin_2)
- new net In b 1: J6.4 (Pin_4)
- new net In b 2: J6.6 (Pin_6)
- new net In b 3: J6.8 (Pin_8)
- new net In c 0: J6.12 (Pin_12)
- new net In c 1: J6.14 (Pin_14)
- new net In c 2: J6.16 (Pin_16)
- new net In c 3: J6.18 (Pin_18)
- new net In c 4: J6.20 (Pin_20)
- new net In c 5: J6.22 (Pin_22)
- new net In c 6: J6.24 (Pin_24)
- new net In c 7: J6.26 (Pin_26)
- new net In d 0: J6.11 (Pin_11)
- new net In d 1: J6.13 (Pin_13)
- new net In d 2: J6.15 (Pin_15)
- new net In d 3: J6.17 (Pin_17)
- new net In d 4: J6.19 (Pin_19)
- new net In d 5: J6.21 (Pin_21)
- new net In d 6: J6.23 (Pin_23)
- new net In d 7: J6.25 (Pin_25)
- new net Out  A: J6.9 (Pin_9)
- new net Out  B: J6.10 (Pin_10)
- new net Out  C: J6.28 (Pin_28)
- new net Out  D: J6.27 (Pin_27)
- new net Out A: J5.13 (Pin_13)
- new net Out B: J5.12 (Pin_12)
- new net Out C: J5.25 (Pin_25)
- new net Out D: J5.26 (Pin_26)
- new net SJ A: J5.11 (Pin_11)
- new net SJ B: J5.14 (Pin_14)
- new net SJ C: J5.27 (Pin_27)
- new net SJ D: J5.28 (Pin_28)
Other:
- added sheet Inverting Summer 4x11SJ (Inverting Summer 4x11SJ.kicad_sch)
- added sheet Inverting Summer 8-2 4-2 (Inverting Summer 8-2 4-2.kicad_sch)
- moved on the sheet: J1, J2, J3, J4

Commit message: update layount
Parts:
- added J7: Conn_02x14_Odd_Even, Connector_PinHeader_2.54mm:PinHeader_2x14_P2.54mm_Vertical, symbol Connector_Generic:Conn_02x14_Odd_Even
Connections:
- new net Buffer In 0: J7.1 (Pin_1)
- new net Buffer In 1: J7.3 (Pin_3)
- new net Buffer In 10: J7.21 (Pin_21)
- new net Buffer In 11: J7.23 (Pin_23)
- new net Buffer In 2: J7.5 (Pin_5)
- new net Buffer In 3: J7.7 (Pin_7)
- new net Buffer In 4: J7.9 (Pin_9)
- new net Buffer In 5: J7.11 (Pin_11)
- new net Buffer In 6: J7.13 (Pin_13)
- new net Buffer In 7: J7.15 (Pin_15)
- new net Buffer In 8: J7.17 (Pin_17)
- new net Buffer In 9: J7.19 (Pin_19)
- new net Buffer Out 0: J7.2 (Pin_2)
- new net Buffer Out 1: J7.4 (Pin_4)
- new net Buffer Out 10: J7.22 (Pin_22)
- new net Buffer Out 11: J7.24 (Pin_24)
- new net Buffer Out 2: J7.6 (Pin_6)
- new net Buffer Out 3: J7.8 (Pin_8)
- new net Buffer Out 4: J7.10 (Pin_10)
- new net Buffer Out 5: J7.12 (Pin_12)
- new net Buffer Out 6: J7.14 (Pin_14)
- new net Buffer Out 7: J7.16 (Pin_16)
- new net Buffer Out 8: J7.18 (Pin_18)
- new net Buffer Out 9: J7.20 (Pin_20)
- no-connect marks 12 -> 16
Other:
- added sheet Buffer Follower 0 (BufferFollower.kicad_sch)
- added sheet Buffer Follower 1 (BufferFollower.kicad_sch)
- added sheet Buffer Follower 2 (BufferFollower.kicad_sch)
- title: Logarithmic Amplifier -> Analog Computer 
- moved on the sheet: J1, J2, J4, J5, J6

Commit message: update analog computer layout
Connections:
- net VSS is gone; now on net GND: J4.1 (Pin_1)
- net GND: no longer J4.3 (Pin_3)
- new net VDD: J4.3 (Pin_3)
Other:
- title: Analog Computer  -> Analog Computer
Changed lines of the file:
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@@
   (paper "A4")
   (title_block
-    (title "Analog Computer ")
+    (title "Analog Computer")
     (date "2023-03-08")
     (rev "v1")
@@
     )
   )
-  (symbol (lib_id "power:GND") (at 223.52 123.19 0) (unit 1)
+  (symbol (lib_id "power:VDD") (at 223.52 123.19 180) (unit 1)
     (in_bom yes) (on_board yes) (dnp no) (fields_autoplaced)
-    (property "Reference" "#PWR030" (at 223.52 129.54 0)
+    (property "Reference" "#PWR030" (at 223.52 116.84 0)
       (effects (font (size 1.27 1.27)) hide)
     )
@@
     )
   )
-  (symbol (lib_id "power:VSS") (at 220.98 104.14 0) (unit 1)
+  (symbol (lib_id "power:GND") (at 220.98 104.14 180) (unit 1)
     (in_bom yes) (on_board yes) (dnp no) (fields_autoplaced)
-    (property "Reference" "#PWR029" (at 220.98 107.95 0)
+    (property "Reference" "#PWR029" (at 220.98 100.33 0)
       (effects (font (size 1.27 1.27)) hide)
     )
