File: circuits/AnalogCalculator/AnalogComputer/Inverting Summer 4x11SJ.kicad_sch (KiCad schematic)
At the start: 9 parts, among them U10 LM324

Commit message: update layount
Parts:
- R49, R50, R51, R52: footprint Resistor_THT_US_AKL:R_Box_L8.4mm_W2.5mm_P5.08mm -> Resistor_THT:R_Axial_DIN0204_L3.6mm_D1.6mm_P2.54mm_Vertical
- RN1, RN2, RN3, RN4: footprint Resistor_THT_US_AKL:R_Array_SIP5_BigPads -> Resistor_THT:R_Array_SIP5
- U10: footprint (none) -> Package_DIP:DIP-14_W7.62mm_Socket
Changed lines of the file:
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@@
       (effects (font (size 1.27 1.27)))
     )
-    (property "Footprint" "Resistor_THT_US_AKL:R_Box_L8.4mm_W2.5mm_P5.08mm" (at 81.28 130.81 0)
+    (property "Footprint" "Resistor_THT:R_Axial_DIN0204_L3.6mm_D1.6mm_P2.54mm_Vertical" (at 81.28 130.81 0)
       (effects (font (size 1.27 1.27)) hide)
     )
@@
       (effects (font (size 1.27 1.27)))
     )
-    (property "Footprint" "" (at 90.17 64.77 0)
+    (property "Footprint" "Package_DIP:DIP-14_W7.62mm_Socket" (at 90.17 64.77 0)
       (effects (font (size 1.27 1.27)) hide)
     )
@@
       (effects (font (size 1.27 1.27)))
     )
-    (property "Footprint" "" (at 90.17 120.65 0)
+    (property "Footprint" "Package_DIP:DIP-14_W7.62mm_Socket" (at 90.17 120.65 0)
       (effects (font (size 1.27 1.27)) hide)
     )
@@
       (effects (font (size 1.27 1.27)))
     )
-    (property "Footprint" "Resistor_THT_US_AKL:R_Array_SIP5_BigPads" (at 58.42 64.77 0)
+    (property "Footprint" "Resistor_THT:R_Array_SIP5" (at 58.42 64.77 0)
       (effects (font (size 1.27 1.27)) hide)
     )
@@
       (effects (font (size 1.27 1.27)))
     )
-    (property "Footprint" "Resistor_THT_US_AKL:R_Array_SIP5_BigPads" (at 58.42 120.65 0)
+    (property "Footprint" "Resistor_THT:R_Array_SIP5" (at 58.42 120.65 0)
       (effects (font (size 1.27 1.27)) hide)
     )
@@
       (effects (font (size 1.27 1.27)))
     )
-    (property "Footprint" "Resistor_THT_US_AKL:R_Box_L8.4mm_W2.5mm_P5.08mm" (at 81.28 46.99 0)
+    (property "Footprint" "Resistor_THT:R_Axial_DIN0204_L3.6mm_D1.6mm_P2.54mm_Vertical" (at 81.28 46.99 0)
       (effects (font (size 1.27 1.27)) hide)
     )
@@
       (effects (font (size 1.27 1.27)))
     )
-    (property "Footprint" "Resistor_THT_US_AKL:R_Array_SIP5_BigPads" (at 58.42 36.83 0)
+    (property "Footprint" "Resistor_THT:R_Array_SIP5" (at 58.42 36.83 0)
       (effects (font (size 1.27 1.27)) hide)
     )
@@
       (effects (font (size 1.27 1.27)))
     )
-    (property "Footprint" "Resistor_THT_US_AKL:R_Array_SIP5_BigPads" (at 58.42 92.71 0)
+    (property "Footprint" "Resistor_THT:R_Array_SIP5" (at 58.42 92.71 0)
       (effects (font (size 1.27 1.27)) hide)
     )
@@
       (effects (font (size 1.27 1.27)))
     )
-    (property "Footprint" "Resistor_THT_US_AKL:R_Box_L8.4mm_W2.5mm_P5.08mm" (at 81.28 102.87 0)
+    (property "Footprint" "Resistor_THT:R_Axial_DIN0204_L3.6mm_D1.6mm_P2.54mm_Vertical" (at 81.28 102.87 0)
       (effects (font (size 1.27 1.27)) hide)
     )
@@
       (effects (font (size 1.27 1.27)))
     )
-    (property "Footprint" "Resistor_THT_US_AKL:R_Box_L8.4mm_W2.5mm_P5.08mm" (at 81.28 74.93 0)
+    (property "Footprint" "Resistor_THT:R_Axial_DIN0204_L3.6mm_D1.6mm_P2.54mm_Vertical" (at 81.28 74.93 0)
       (effects (font (size 1.27 1.27)) hide)
     )
@@
       (effects (font (size 1.27 1.27)))
     )
-    (property "Footprint" "" (at 90.17 92.71 0)
+    (property "Footprint" "Package_DIP:DIP-14_W7.62mm_Socket" (at 90.17 92.71 0)
       (effects (font (size 1.27 1.27)) hide)
     )
@@
       (effects (font (size 1.27 1.27)) (justify left))
     )
-    (property "Footprint" "" (at 140.97 81.28 0)
+    (property "Footprint" "Package_DIP:DIP-14_W7.62mm_Socket" (at 140.97 81.28 0)
       (effects (font (size 1.27 1.27)) hide)
     )
@@
       (effects (font (size 1.27 1.27)))
     )
-    (property "Footprint" "" (at 90.17 36.83 0)
-      (effects (font (size 1.27 1.27)) hide)
-    )
+    (property "Footprint" "Package_DIP:DIP-14_W7.62mm_Socket" (at 90.17 36.83 0)
+      (effects (font (size 1.27 1.27)) hide)
+    )

Commit message: update analog computer layout
Connections:
- net VSS is gone; now on net GND: U10.11 (V-)
- net GND: no longer U10.10 (+), U10.12 (+), U10.3 (+), U10.5 (+)
- new net VDD: U10.10 (+), U10.12 (+), U10.3 (+), U10.5 (+)
Other:
- company: Out-of-Band Development -> Out-of-band Development, LLC
- title: Inverting Summer with 4x10k + 1x1k + SJ -> Analog Computer
Changed lines of the file:
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@@
   (paper "A4")
   (title_block
-    (title "Inverting Summer with 4x10k + 1x1k + SJ")
+    (title "Analog Computer")
     (date "2023-03-08")
-    (company "Out-of-Band Development")
+    (rev "v1")
+    (company "Out-of-band Development, LLC")
     (comment 1 "Matthew Whited")
+    (comment 2 "Inverting Summing Amplifier")
+    (comment 3 "4x10k, 1x1k with Summing Junction and No Feedback")
   )
   (junction (at 77.47 97.79) (diameter 0) (color 0 0 0 0)
@@
     )
   )
-  (symbol (lib_id "power:GND") (at 81.28 36.83 0) (unit 1)
+  (symbol (lib_id "power:VDD") (at 81.28 36.83 0) (unit 1)
     (in_bom yes) (on_board yes) (dnp no) (fields_autoplaced)
     (property "Reference" "#PWR031" (at 81.28 43.18 0)
@@
     )
   )
-  (symbol (lib_id "power:GND") (at 81.28 92.71 0) (unit 1)
+  (symbol (lib_id "power:VDD") (at 81.28 92.71 0) (unit 1)
     (in_bom yes) (on_board yes) (dnp no) (fields_autoplaced)
     (property "Reference" "#PWR033" (at 81.28 99.06 0)
@@
     )
   )
-  (symbol (lib_id "power:GND") (at 81.28 120.65 0) (unit 1)
+  (symbol (lib_id "power:VDD") (at 81.28 120.65 0) (unit 1)
     (in_bom yes) (on_board yes) (dnp no) (fields_autoplaced)
     (property "Reference" "#PWR034" (at 81.28 127 0)
@@
     )
   )
-  (symbol (lib_id "power:VSS") (at 139.7 96.52 180) (unit 1)
+  (symbol (lib_id "power:GND") (at 139.7 96.52 180) (unit 1)
     (in_bom yes) (on_board yes) (dnp no) (fields_autoplaced)
     (property "Reference" "#PWR036" (at 139.7 92.71 0)
@@
     )
   )
-  (symbol (lib_id "power:GND") (at 81.28 64.77 0) (unit 1)
+  (symbol (lib_id "power:VDD") (at 81.28 64.77 0) (unit 1)
     (in_bom yes) (on_board yes) (dnp no) (fields_autoplaced)
     (property "Reference" "#PWR032" (at 81.28 71.12 0)
