File: circuits/AnalogCalculator/AnalogComputer/Logarithmic Amplifier.kicad_sch (KiCad schematic)
At the start: 9 parts, among them U1 LM324

Commit message: update circuits
Connections:
- net +12V renamed VCC
- net -12V renamed VSS
Changed lines of the file:
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@@
+    (stroke (width 0) (type default))
+  )
+  (wire (pts (xy 172.72 95.25) (xy 172.72 106.68))
     (stroke (width 0) (type default))
   )
@@
   )
   (wire (pts (xy 80.01 116.84) (xy 77.47 116.84))
-    (stroke (width 0) (type default))
-  )
-  (wire (pts (xy 172.72 95.25) (xy 172.72 106.68))
     (stroke (width 0) (type default))
   )
@@
     )
   )
-  (symbol (lib_id "power:-12V") (at 187.96 95.25 0) (unit 1)
-    (in_bom yes) (on_board yes) (dnp no) (fields_autoplaced)
-    (property "Reference" "#PWR02" (at 187.96 92.71 0)
-      (effects (font (size 1.27 1.27)) hide)
-    )
-    (property "Value" "-12V" (at 187.96 91.6742 0)
-      (effects (font (size 1.27 1.27)))
-    )
-    (property "Footprint" "" (at 187.96 95.25 0)
-      (effects (font (size 1.27 1.27)) hide)
-    )
-    (property "Datasheet" "" (at 187.96 95.25 0)
-      (effects (font (size 1.27 1.27)) hide)
-    )
-    (pin "1")
-    (instances
-      (project "AnalogComputer"
-        (path "/923be781-3164-4152-815e-8f20a1ba1c2e/b258d8fb-1fa9-4360-b935-b0ac69a48bdd"
-          (reference "#PWR02") (unit 1)
-        )
-        (path "/923be781-3164-4152-815e-8f20a1ba1c2e/e2f4230b-19f4-4916-8902-56d8b1497f4b"
-          (reference "#PWR011") (unit 1)
-        )
-        (path "/923be781-3164-4152-815e-8f20a1ba1c2e/6e6abdf6-4cd3-46b5-a236-3b3c53ee6c51"
-          (reference "#PWR08") (unit 1)
-        )
-      )
-    )
-  )
   (symbol (lib_id "Amplifier_Operational:LM324") (at 175.26 114.3 0) (unit 5)
     (in_bom yes) (on_board yes) (dnp no) (fields_autoplaced)
@@
     )
   )
+  (symbol (lib_id "power:VCC") (at 172.72 95.25 0) (unit 1)
+    (in_bom yes) (on_board yes) (dnp no) (fields_autoplaced)
+    (property "Reference" "#PWR01" (at 172.72 99.06 0)
+      (effects (font (size 1.27 1.27)) hide)
+    )
+    (property "Value" "VCC" (at 172.72 91.7481 0)
+      (effects (font (size 1.27 1.27)))
+    )
+    (property "Footprint" "" (at 172.72 95.25 0)
+      (effects (font (size 1.27 1.27)) hide)
+    )
+    (property "Datasheet" "" (at 172.72 95.25 0)
+      (effects (font (size 1.27 1.27)) hide)
+    )
+    (pin "1")
+    (instances
+      (project "AnalogComputer"
+        (path "/923be781-3164-4152-815e-8f20a1ba1c2e/b258d8fb-1fa9-4360-b935-b0ac69a48bdd"
+          (reference "#PWR01") (unit 1)
+        )
+        (path "/923be781-3164-4152-815e-8f20a1ba1c2e/6e6abdf6-4cd3-46b5-a236-3b3c53ee6c51"
+          (reference "#PWR02") (unit 1)
+        )
+        (path "/923be781-3164-4152-815e-8f20a1ba1c2e/e2f4230b-19f4-4916-8902-56d8b1497f4b"
+          (reference "#PWR07") (unit 1)
+        )
+      )
+    )
+  )
   (symbol (lib_id "pspice:DIODE") (at 144.78 127 0) (unit 1)
     (in_bom yes) (on_board yes) (dnp no) (fields_autoplaced)
@@
     )
   )
-  (symbol (lib_id "power:+12V") (at 172.72 95.25 0) (unit 1)
-    (in_bom yes) (on_board yes) (dnp no) (fields_autoplaced)
-    (property "Reference" "#PWR01" (at 172.72 99.06 0)
-      (effects (font (size 1.27 1.27)) hide)
-    )
-    (property "Value" "+12V" (at 172.72 91.6742 0)
-      (effects (font (size 1.27 1.27)))
-    )
-    (property "Footprint" "" (at 172.72 95.25 0)
-      (effects (font (size 1.27 1.27)) hide)
-    )
-    (property "Datasheet" "" (at 172.72 95.25 0)
-      (effects (font (size 1.27 1.27)) hide)
-    )
-    (pin "1")
-    (instances
-      (project "AnalogComputer"
-        (path "/923be781-3164-4152-815e-8f20a1ba1c2e/b258d8fb-1fa9-4360-b935-b0ac69a48bdd"
-          (reference "#PWR01") (unit 1)
-        )
-        (path "/923be781-3164-4152-815e-8f20a1ba1c2e/e2f4230b-19f4-4916-8902-56d8b1497f4b"
-          (reference "#PWR010") (unit 1)
-        )
-        (path "/923be781-3164-4152-815e-8f20a1ba1c2e/6e6abdf6-4cd3-46b5-a236-3b3c53ee6c51"
-          (reference "#PWR07") (unit 1)
-        )
-      )
-    )
-  )
   (symbol (lib_id "Device:R") (at 50.8 132.08 0) (unit 1)
     (in_bom yes) (on_board yes) (dnp no) (fields_autoplaced)
@@
         )
       )
+    )
+  )
+  (symbol (lib_id "power:VSS") (at 187.96 95.25 0) (unit 1)
+    (in_bom yes) (on_board yes) (dnp no) (fields_autoplaced)
+    (property "Reference" "#PWR08" (at 187.96 99.06 0)
+      (effects (font (size 1.27 1.27)) hide)
+    )
+    (property "Value" "VSS" (at 187.96 91.7481 0)
+      (effects (font (size 1.27 1.27)))
+    )
+    (property "Footprint" "" (at 187.96 95.25 0)
+      (effects (font (size 1.27 1.27)) hide)
+    )
+    (property "Datasheet" "" (at 187.96 95.25 0)
+      (effects (font (size 1.27 1.27)) hide)
+    )
+    (pin "1")
+    (instances
+      (project "AnalogComputer"
+        (path "/923be781-3164-4152-815e-8f20a1ba1c2e/b258d8fb-1fa9-4360-b935-b0ac69a48bdd"
+          (reference "#PWR08") (unit 1)
+        )
+        (path "/923be781-3164-4152-815e-8f20a1ba1c2e/6e6abdf6-4cd3-46b5-a236-3b3c53ee6c51"
+          (reference "#PWR010") (unit 1)
+        )
+        (path "/923be781-3164-4152-815e-8f20a1ba1c2e/e2f4230b-19f4-4916-8902-56d8b1497f4b"
+          (reference "#PWR011") (unit 1)
+        )
+      )

Commit message: update analog computer layout
Connections:
- net VSS is gone; now on net GND: U1.11 (V-)
- net GND: no longer U1.10 (+), U1.12 (+), U1.3 (+), U1.5 (+)
- new net VDD: U1.10 (+), U1.12 (+), U1.3 (+), U1.5 (+)
Other:
- title: Logarithmic Amplifier -> Analog Computer
Changed lines of the file:
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@@
   (paper "A4")
   (title_block
-    (title "Logarithmic Amplifier")
-    (date "2023-03-06")
+    (title "Analog Computer")
+    (date "2023-03-08")
     (rev "v1")
     (company "Out-of-band Development, LLC")
     (comment 1 "Matthew Whited")
+    (comment 2 "Logarithmic Amplifer")
   )
   (junction (at 50.8 96.52) (diameter 0) (color 0 0 0 0)
@@
     )
   )
-  (symbol (lib_id "power:GND") (at 39.37 96.52 0) (unit 1)
+  (symbol (lib_id "power:VDD") (at 39.37 96.52 0) (unit 1)
     (in_bom yes) (on_board yes) (dnp no) (fields_autoplaced)
     (property "Reference" "#PWR03" (at 39.37 102.87 0)
@@
     )
   )
-  (symbol (lib_id "power:VSS") (at 187.96 95.25 0) (unit 1)
+  (symbol (lib_id "power:GND") (at 187.96 95.25 0) (unit 1)
     (in_bom yes) (on_board yes) (dnp no) (fields_autoplaced)
     (property "Reference" "#PWR08" (at 187.96 99.06 0)
