File: circuits/AnalogCalculator/SimpleOpAmp/Simple OpAmp/Simple OpAmp.kicad_pcb (KiCad board)
At the start: 2 copper layers, 137 x 125.5 mm, 181 parts, among them J1 Conn_02x10_Odd_Even, J2 Conn_01x03_Pin, J3 Conn_02x10_Odd_Even, J4 Conn_02x10_Odd_Even, J5 Conn_02x10_Odd_Even, J6 Conn_02x10_Odd_Even, J7 Conn_02x10_Odd_Even, J8 Conn_02x10_Odd_Even, J9 Conn_02x10_Odd_Even, U1 Opamp_Quad, U2 Opamp_Quad, U3 Opamp_Quad, U4 Opamp_Quad

Commit message: update
Parts:
- removed C1, C2, C3, C4: C_Trim_Differential, Potentiometer_THT:Potentiometer_Runtron_RM-065_Vertical
- removed H2, H3, H4, H5, H6, H7, H8: MountingHole_3mm_Pad_TopBottom, MountingHole:MountingHole_3mm_Pad_TopBottom
- removed J1, J4: Conn_02x10_Odd_Even, Connector_PinSocket_2.54mm:PinSocket_2x10_P2.54mm_Vertical
- removed J2: Conn_01x03_Pin, Connector_PinHeader_2.54mm:PinHeader_1x03_P2.54mm_Vertical
- removed RV1, RV10, RV11, RV12, RV13, RV14, RV15, RV16, RV17, RV18, RV19, RV2, RV20, RV21, RV22, RV23, RV24, RV25, RV26, RV27, RV28, RV29, RV3, RV30, RV31, RV32, RV33, RV34, RV35, RV36, RV4, RV5, RV6, RV7, RV8, RV9: R_Potentiometer_US, Potentiometer_THT:Potentiometer_Bourns_3266Y_Vertical
- removed U1: Opamp_Quad, Package_DIP:DIP-14_W7.62mm_Socket_LongPads
- added C17: C_Trim_Differential, Potentiometer_THT:Potentiometer_Runtron_RM-065_Vertical, F.Cu at (92.5, 166.8)
- added C18: C_Trim_Differential, Potentiometer_THT:Potentiometer_Runtron_RM-065_Vertical, F.Cu at (100.6, 166.8)
- added C19: C_Trim_Differential, Potentiometer_THT:Potentiometer_Runtron_RM-065_Vertical, F.Cu at (108.7, 166.8)
- added C20: C_Trim_Differential, Potentiometer_THT:Potentiometer_Runtron_RM-065_Vertical, F.Cu at (116.8, 166.8)
- added J10: Conn_02x10_Odd_Even, Connector_PinSocket_2.54mm:PinSocket_2x10_P2.54mm_Vertical, F.Cu at (74.9, 167.1)
- added J12: Conn_02x10_Odd_Even, Connector_PinSocket_2.54mm:PinSocket_2x10_P2.54mm_Vertical, F.Cu at (128.2, 167.1)
- added J13: Conn_02x10_Odd_Even, Connector_PinSocket_2.54mm:PinSocket_2x10_P2.54mm_Vertical, F.Cu at (135.4, 167.1)
- added RV145: R_Potentiometer_US, Potentiometer_THT:Potentiometer_Bourns_3266Y_Vertical, F.Cu at (97.6, 131.1)
- added RV146: R_Potentiometer_US, Potentiometer_THT:Potentiometer_Bourns_3266Y_Vertical, F.Cu at (97.6, 137.2)
- added RV147: R_Potentiometer_US, Potentiometer_THT:Potentiometer_Bourns_3266Y_Vertical, F.Cu at (97.6, 143.3)
- added RV148: R_Potentiometer_US, Potentiometer_THT:Potentiometer_Bourns_3266Y_Vertical, F.Cu at (97.6, 149.4)
- added RV149: R_Potentiometer_US, Potentiometer_THT:Potentiometer_Bourns_3266Y_Vertical, F.Cu at (97.6, 155.5)
- added RV150: R_Potentiometer_US, Potentiometer_THT:Potentiometer_Bourns_3266Y_Vertical, F.Cu at (97.6, 161.6)
- added RV151: R_Potentiometer_US, Potentiometer_THT:Potentiometer_Bourns_3266Y_Vertical, F.Cu at (105.9, 131.1)
- added RV152: R_Potentiometer_US, Potentiometer_THT:Potentiometer_Bourns_3266Y_Vertical, F.Cu at (105.9, 137.2)
- added RV153: R_Potentiometer_US, Potentiometer_THT:Potentiometer_Bourns_3266Y_Vertical, F.Cu at (105.9, 143.3)
- added RV154: R_Potentiometer_US, Potentiometer_THT:Potentiometer_Bourns_3266Y_Vertical, F.Cu at (105.9, 149.4)
- added RV155: R_Potentiometer_US, Potentiometer_THT:Potentiometer_Bourns_3266Y_Vertical, F.Cu at (105.9, 155.5)
- added RV156: R_Potentiometer_US, Potentiometer_THT:Potentiometer_Bourns_3266Y_Vertical, F.Cu at (105.9, 161.6)
- added RV157: R_Potentiometer_US, Potentiometer_THT:Potentiometer_Bourns_3266Y_Vertical, F.Cu at (114.2, 131.1)
- added RV158: R_Potentiometer_US, Potentiometer_THT:Potentiometer_Bourns_3266Y_Vertical, F.Cu at (114.2, 137.2)
- added RV159: R_Potentiometer_US, Potentiometer_THT:Potentiometer_Bourns_3266Y_Vertical, F.Cu at (114.2, 143.3)
- added RV160: R_Potentiometer_US, Potentiometer_THT:Potentiometer_Bourns_3266Y_Vertical, F.Cu at (114.2, 149.4)
- added RV161: R_Potentiometer_US, Potentiometer_THT:Potentiometer_Bourns_3266Y_Vertical, F.Cu at (114.2, 155.5)
- added RV162: R_Potentiometer_US, Potentiometer_THT:Potentiometer_Bourns_3266Y_Vertical, F.Cu at (114.2, 161.6)
- added RV163: R_Potentiometer_US, Potentiometer_THT:Potentiometer_Bourns_3266Y_Vertical, F.Cu at (122.5, 131.1)
- added RV164: R_Potentiometer_US, Potentiometer_THT:Potentiometer_Bourns_3266Y_Vertical, F.Cu at (122.5, 137.2)
- added RV165: R_Potentiometer_US, Potentiometer_THT:Potentiometer_Bourns_3266Y_Vertical, F.Cu at (122.5, 143.3)
- added RV166: R_Potentiometer_US, Potentiometer_THT:Potentiometer_Bourns_3266Y_Vertical, F.Cu at (122.5, 149.4)
- added RV167: R_Potentiometer_US, Potentiometer_THT:Potentiometer_Bourns_3266Y_Vertical, F.Cu at (122.5, 155.5)
- added RV168: R_Potentiometer_US, Potentiometer_THT:Potentiometer_Bourns_3266Y_Vertical, F.Cu at (122.5, 161.6)
- added RV169: R_Potentiometer_US, Potentiometer_THT:Potentiometer_Bourns_3266Y_Vertical, F.Cu at (130.8, 131.1)
- added RV170: R_Potentiometer_US, Potentiometer_THT:Potentiometer_Bourns_3266Y_Vertical, F.Cu at (130.8, 137.2)
- added RV171: R_Potentiometer_US, Potentiometer_THT:Potentiometer_Bourns_3266Y_Vertical, F.Cu at (130.8, 143.3)
- added RV172: R_Potentiometer_US, Potentiometer_THT:Potentiometer_Bourns_3266Y_Vertical, F.Cu at (130.8, 149.4)
- added RV173: R_Potentiometer_US, Potentiometer_THT:Potentiometer_Bourns_3266Y_Vertical, F.Cu at (130.8, 155.5)
- added RV174: R_Potentiometer_US, Potentiometer_THT:Potentiometer_Bourns_3266Y_Vertical, F.Cu at (130.8, 161.6)
- added RV175: R_Potentiometer_US, Potentiometer_THT:Potentiometer_Bourns_3266Y_Vertical, F.Cu at (139.1, 131.1)
- added RV176: R_Potentiometer_US, Potentiometer_THT:Potentiometer_Bourns_3266Y_Vertical, F.Cu at (139.1, 137.2)
- added RV177: R_Potentiometer_US, Potentiometer_THT:Potentiometer_Bourns_3266Y_Vertical, F.Cu at (139.1, 143.3)
- added RV178: R_Potentiometer_US, Potentiometer_THT:Potentiometer_Bourns_3266Y_Vertical, F.Cu at (139.1, 149.4)
- added RV179: R_Potentiometer_US, Potentiometer_THT:Potentiometer_Bourns_3266Y_Vertical, F.Cu at (139.1, 155.5)
- added RV180: R_Potentiometer_US, Potentiometer_THT:Potentiometer_Bourns_3266Y_Vertical, F.Cu at (139.1, 161.6)
- added U5: Opamp_Quad, Package_DIP:DIP-14_W7.62mm_Socket_LongPads, F.Cu at (139.7, 166.8)
- J3: value Conn_02x10_Odd_Even -> Conn_01x03_Pin; footprint Connector_PinSocket_2.54mm:PinSocket_2x10_P2.54mm_Vertical -> Connector_PinHeader_2.54mm:PinHeader_1x03_P2.54mm_Vertical
- moved RV89 324.9 mm to (-166.5, 5.50), turned to 0 degrees
- moved RV86 301.5 mm to (-130.5, -16.4), turned to 0 degrees
- moved RV76 297.3 mm to (-152.0, -4.00), turned to 0 degrees
- moved RV80 296.8 mm to (-146.4, -16.5), turned to 0 degrees
- moved RV75 287.4 mm to (-128.5, -26.0), turned to 0 degrees
- moved RV84 277.0 mm to (-150.5, 7.00), turned to 0 degrees
- moved C9 274.0 mm to (-148.5, -35.3)
- moved RV82 273.7 mm to (-138.5, -3.50), turned to 0 degrees
- moved J7 273.7 mm to (-104.5, -23.3), turned to 0 degrees
- moved RV73 268.4 mm to (-129.0, -45.3), turned to 0 degrees
- moved RV78 261.8 mm to (-130.0, -4.50), turned to 0 degrees
- moved RV85 243.6 mm to (-55.9, -48.0), turned to 0 degrees
- moved C11 236.6 mm to (-150.0, 33.0)
- moved RV79 234.6 mm to (-78.5, -38.8), turned to 0 degrees
- moved RV74 229.3 mm to (-78.5, -46.3), turned to 0 degrees
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Connections:
- C10 pad 1: Net-(J4-Pin_4) -> Net-(J7-Pin_17)
- C10 pad 2: Net-(J4-Pin_2) -> Net-(J7-Pin_19)
- C10 pad 3: unconnected-(C3-Pad3) -> unconnected-(C10-Pad3)
- C11 pad 1: Net-(J3-Pin_4) -> Net-(J8-Pin_4)
- C11 pad 2: Net-(J3-Pin_2) -> Net-(J8-Pin_2)
- C11 pad 3: unconnected-(C2-Pad3) -> unconnected-(C11-Pad3)
- C12 pad 1: Net-(J4-Pin_17) -> Net-(J8-Pin_17)
- C12 pad 2: Net-(J4-Pin_19) -> Net-(J8-Pin_19)
- C12 pad 3: unconnected-(C4-Pad3) -> unconnected-(C12-Pad3)
- C13 pad 1: Net-(J3-Pin_17) -> Net-(J9-Pin_4)
- C13 pad 2: Net-(J3-Pin_19) -> Net-(J9-Pin_2)
- C13 pad 3: unconnected-(C1-Pad3) -> unconnected-(C13-Pad3)
- C14 pad 1: Net-(J3-Pin_4) -> Net-(J9-Pin_17)
- C14 pad 2: Net-(J3-Pin_2) -> Net-(J9-Pin_19)
- C14 pad 3: unconnected-(C2-Pad3) -> unconnected-(C14-Pad3)
- C15 pad 1: Net-(J4-Pin_4) -> Net-(J10-Pin_4)
- C15 pad 2: Net-(J4-Pin_2) -> Net-(J10-Pin_2)
- C15 pad 3: unconnected-(C3-Pad3) -> unconnected-(C15-Pad3)
- C16 pad 1: Net-(J4-Pin_17) -> Net-(J10-Pin_17)
- C16 pad 2: Net-(J4-Pin_19) -> Net-(J10-Pin_19)
- C16 pad 3: unconnected-(C4-Pad3) -> unconnected-(C16-Pad3)
- C5 pad 1: Net-(J4-Pin_17) -> Net-(J5-Pin_4)
- C5 pad 2: Net-(J4-Pin_19) -> Net-(J5-Pin_2)
- C5 pad 3: unconnected-(C4-Pad3) -> unconnected-(C5-Pad3)
- C6 pad 1: Net-(J4-Pin_4) -> Net-(J5-Pin_17)
- C6 pad 2: Net-(J4-Pin_2) -> Net-(J5-Pin_19)
- C6 pad 3: unconnected-(C3-Pad3) -> unconnected-(C6-Pad3)
- C7 pad 1: Net-(J3-Pin_17) -> Net-(J6-Pin_4)
- C7 pad 2: Net-(J3-Pin_19) -> Net-(J6-Pin_2)
- C7 pad 3: unconnected-(C1-Pad3) -> unconnected-(C7-Pad3)
- C8 pad 1: Net-(J3-Pin_4) -> Net-(J6-Pin_17)
- C8 pad 2: Net-(J3-Pin_2) -> Net-(J6-Pin_19)
- C8 pad 3: unconnected-(C2-Pad3) -> unconnected-(C8-Pad3)
- C9 pad 1: Net-(J4-Pin_17) -> Net-(J7-Pin_4)
- C9 pad 2: Net-(J4-Pin_19) -> Net-(J7-Pin_2)
- C9 pad 3: unconnected-(C4-Pad3) -> unconnected-(C9-Pad3)
- J3 pad 1: Net-(J4-Pin_1) -> +15V
- J3 pad 2: Net-(J4-Pin_2) -> GND
- J3 pad 3: Net-(J4-Pin_3) -> -15V
- J5 pad 1: Net-(J4-Pin_1) -> Net-(J5-Pin_1)
- J5 pad 10: Net-(J4-Pin_10) -> Net-(J5-Pin_10)
- J5 pad 11: Net-(J4-Pin_11) -> Net-(J5-Pin_11)
- J5 pad 12: Net-(J4-Pin_12) -> Net-(J5-Pin_12)
- J5 pad 13: Net-(J4-Pin_13) -> Net-(J5-Pin_13)
- J5 pad 14: Net-(J4-Pin_14) -> Net-(J5-Pin_14)
- J5 pad 15: Net-(J4-Pin_15) -> Net-(J5-Pin_15)
- J5 pad 16: Net-(J4-Pin_16) -> Net-(J5-Pin_16)
- J5 pad 17: Net-(J4-Pin_17) -> Net-(J5-Pin_17)
- J5 pad 18: Net-(J4-Pin_18) -> Net-(J5-Pin_18)
- J5 pad 19: Net-(J4-Pin_19) -> Net-(J5-Pin_19)
- J5 pad 2: Net-(J4-Pin_2) -> Net-(J5-Pin_2)
- J5 pad 20: Net-(J4-Pin_20) -> Net-(J5-Pin_20)
- J5 pad 3: Net-(J4-Pin_3) -> Net-(J5-Pin_3)
- J5 pad 4: Net-(J4-Pin_4) -> Net-(J5-Pin_4)
- J5 pad 5: Net-(J4-Pin_5) -> Net-(J5-Pin_5)
- J5 pad 6: Net-(J4-Pin_6) -> Net-(J5-Pin_6)
- J5 pad 7: Net-(J4-Pin_7) -> Net-(J5-Pin_7)
- J5 pad 8: Net-(J4-Pin_8) -> Net-(J5-Pin_8)
- J5 pad 9: Net-(J4-Pin_9) -> Net-(J5-Pin_9)
- J6 pad 1: Net-(J3-Pin_1) -> Net-(J6-Pin_1)
- J6 pad 10: Net-(J3-Pin_10) -> Net-(J6-Pin_10)
- J6 pad 11: Net-(J3-Pin_11) -> Net-(J6-Pin_11)
- J6 pad 12: Net-(J3-Pin_12) -> Net-(J6-Pin_12)
- J6 pad 13: Net-(J3-Pin_13) -> Net-(J6-Pin_13)
- J6 pad 14: Net-(J3-Pin_14) -> Net-(J6-Pin_14)
- J6 pad 15: Net-(J3-Pin_15) -> Net-(J6-Pin_15)
- J6 pad 16: Net-(J3-Pin_16) -> Net-(J6-Pin_16)
- J6 pad 17: Net-(J3-Pin_17) -> Net-(J6-Pin_17)
- J6 pad 18: Net-(J3-Pin_18) -> Net-(J6-Pin_18)
- J6 pad 19: Net-(J3-Pin_19) -> Net-(J6-Pin_19)
- J6 pad 2: Net-(J3-Pin_2) -> Net-(J6-Pin_2)
- J6 pad 20: Net-(J3-Pin_20) -> Net-(J6-Pin_20)
- J6 pad 3: Net-(J3-Pin_3) -> Net-(J6-Pin_3)
- J6 pad 4: Net-(J3-Pin_4) -> Net-(J6-Pin_4)
- J6 pad 5: Net-(J3-Pin_5) -> Net-(J6-Pin_5)
- J6 pad 6: Net-(J3-Pin_6) -> Net-(J6-Pin_6)
- J6 pad 7: Net-(J3-Pin_7) -> Net-(J6-Pin_7)
- J6 pad 8: Net-(J3-Pin_8) -> Net-(J6-Pin_8)
- J6 pad 9: Net-(J3-Pin_9) -> Net-(J6-Pin_9)
- J7 pad 1: Net-(J4-Pin_1) -> Net-(J7-Pin_1)
- J7 pad 10: Net-(J4-Pin_10) -> Net-(J7-Pin_10)
- J7 pad 11: Net-(J4-Pin_11) -> Net-(J7-Pin_11)
- J7 pad 12: Net-(J4-Pin_12) -> Net-(J7-Pin_12)
- J7 pad 13: Net-(J4-Pin_13) -> Net-(J7-Pin_13)
- J7 pad 14: Net-(J4-Pin_14) -> Net-(J7-Pin_14)
- J7 pad 15: Net-(J4-Pin_15) -> Net-(J7-Pin_15)
- J7 pad 16: Net-(J4-Pin_16) -> Net-(J7-Pin_16)
- J7 pad 17: Net-(J4-Pin_17) -> Net-(J7-Pin_17)
- J7 pad 18: Net-(J4-Pin_18) -> Net-(J7-Pin_18)
- J7 pad 19: Net-(J4-Pin_19) -> Net-(J7-Pin_19)
- J7 pad 2: Net-(J4-Pin_2) -> Net-(J7-Pin_2)
- J7 pad 20: Net-(J4-Pin_20) -> Net-(J7-Pin_20)
- J7 pad 3: Net-(J4-Pin_3) -> Net-(J7-Pin_3)
- J7 pad 4: Net-(J4-Pin_4) -> Net-(J7-Pin_4)
- J7 pad 5: Net-(J4-Pin_5) -> Net-(J7-Pin_5)
- J7 pad 6: Net-(J4-Pin_6) -> Net-(J7-Pin_6)
- J7 pad 7: Net-(J4-Pin_7) -> Net-(J7-Pin_7)
- J7 pad 8: Net-(J4-Pin_8) -> Net-(J7-Pin_8)
- J7 pad 9: Net-(J4-Pin_9) -> Net-(J7-Pin_9)
- J8 pad 1: Net-(J3-Pin_1) -> Net-(J8-Pin_1)
- J8 pad 10: Net-(J3-Pin_10) -> Net-(J8-Pin_10)
- J8 pad 11: Net-(J3-Pin_11) -> Net-(J8-Pin_11)
- J8 pad 12: Net-(J3-Pin_12) -> Net-(J8-Pin_12)
- J8 pad 13: Net-(J3-Pin_13) -> Net-(J8-Pin_13)
- J8 pad 14: Net-(J3-Pin_14) -> Net-(J8-Pin_14)
- J8 pad 15: Net-(J3-Pin_15) -> Net-(J8-Pin_15)
- J8 pad 16: Net-(J3-Pin_16) -> Net-(J8-Pin_16)
- J8 pad 17: Net-(J3-Pin_17) -> Net-(J8-Pin_17)
- J8 pad 18: Net-(J3-Pin_18) -> Net-(J8-Pin_18)
- J8 pad 19: Net-(J3-Pin_19) -> Net-(J8-Pin_19)
- J8 pad 2: Net-(J3-Pin_2) -> Net-(J8-Pin_2)
- J8 pad 20: Net-(J3-Pin_20) -> Net-(J8-Pin_20)
- J8 pad 3: Net-(J3-Pin_3) -> Net-(J8-Pin_3)
- J8 pad 4: Net-(J3-Pin_4) -> Net-(J8-Pin_4)
- J8 pad 5: Net-(J3-Pin_5) -> Net-(J8-Pin_5)
- J8 pad 6: Net-(J3-Pin_6) -> Net-(J8-Pin_6)
- J8 pad 7: Net-(J3-Pin_7) -> Net-(J8-Pin_7)
- J8 pad 8: Net-(J3-Pin_8) -> Net-(J8-Pin_8)
- J8 pad 9: Net-(J3-Pin_9) -> Net-(J8-Pin_9)
- J9 pad 1: Net-(J4-Pin_1) -> Net-(J9-Pin_1)
- J9 pad 10: Net-(J4-Pin_10) -> Net-(J9-Pin_10)
- J9 pad 11: Net-(J4-Pin_11) -> Net-(J9-Pin_11)
- J9 pad 12: Net-(J4-Pin_12) -> Net-(J9-Pin_12)
- J9 pad 13: Net-(J4-Pin_13) -> Net-(J9-Pin_13)
- J9 pad 14: Net-(J4-Pin_14) -> Net-(J9-Pin_14)
- J9 pad 15: Net-(J4-Pin_15) -> Net-(J9-Pin_15)
- J9 pad 16: Net-(J4-Pin_16) -> Net-(J9-Pin_16)
- J9 pad 17: Net-(J4-Pin_17) -> Net-(J9-Pin_17)
- J9 pad 18: Net-(J4-Pin_18) -> Net-(J9-Pin_18)
- J9 pad 19: Net-(J4-Pin_19) -> Net-(J9-Pin_19)
- J9 pad 2: Net-(J4-Pin_2) -> Net-(J9-Pin_2)
- J9 pad 20: Net-(J4-Pin_20) -> Net-(J9-Pin_20)
- J9 pad 3: Net-(J4-Pin_3) -> Net-(J9-Pin_3)
- J9 pad 4: Net-(J4-Pin_4) -> Net-(J9-Pin_4)
- J9 pad 5: Net-(J4-Pin_5) -> Net-(J9-Pin_5)
- J9 pad 6: Net-(J4-Pin_6) -> Net-(J9-Pin_6)
- J9 pad 7: Net-(J4-Pin_7) -> Net-(J9-Pin_7)
- J9 pad 8: Net-(J4-Pin_8) -> Net-(J9-Pin_8)
- J9 pad 9: Net-(J4-Pin_9) -> Net-(J9-Pin_9)
- RV100 pad 1: unconnected-(RV3-Pad1) -> unconnected-(RV100-Pad1)
- RV100 pad 2: Net-(J3-Pin_17) -> Net-(J8-Pin_4)
- RV100 pad 3: Net-(J3-Pin_11) -> Net-(J8-Pin_14)
- RV101 pad 1: unconnected-(RV9-Pad1) -> unconnected-(RV101-Pad1)
- RV101 pad 2: Net-(J3-Pin_17) -> Net-(J8-Pin_17)
- RV101 pad 3: Net-(J3-Pin_13) -> Net-(J8-Pin_9)
- RV102 pad 1: unconnected-(RV14-Pad1) -> unconnected-(RV102-Pad1)
- RV102 pad 2: Net-(J3-Pin_4) -> Net-(J8-Pin_4)
- RV102 pad 3: Net-(J3-Pin_12) -> Net-(J8-Pin_16)
- RV103 pad 1: unconnected-(RV13-Pad1) -> unconnected-(RV103-Pad1)
- RV103 pad 2: Net-(J3-Pin_4) -> Net-(J8-Pin_17)
- RV103 pad 3: Net-(J3-Pin_14) -> Net-(J8-Pin_11)
- RV104 pad 1: unconnected-(RV12-Pad1) -> unconnected-(RV104-Pad1)
- RV104 pad 2: Net-(J3-Pin_4) -> Net-(J8-Pin_4)
- RV104 pad 3: Net-(J3-Pin_16) -> Net-(J8-Pin_18)
- RV105 pad 1: unconnected-(RV1-Pad1) -> unconnected-(RV105-Pad1)
- RV105 pad 2: Net-(J3-Pin_19) -> Net-(J8-Pin_17)
- RV105 pad 3: Net-(J3-Pin_17) -> Net-(J8-Pin_13)
- RV106 pad 1: unconnected-(RV2-Pad1) -> unconnected-(RV106-Pad1)
- RV106 pad 2: Net-(J3-Pin_17) -> Net-(J8-Pin_17)
- RV106 pad 3: Net-(J3-Pin_15) -> Net-(J8-Pin_15)
- RV107 pad 1: unconnected-(RV10-Pad1) -> unconnected-(RV107-Pad1)
- RV107 pad 2: Net-(J3-Pin_4) -> Net-(J8-Pin_4)
- RV107 pad 3: Net-(J3-Pin_20) -> Net-(J8-Pin_20)
- RV108 pad 1: unconnected-(RV11-Pad1) -> unconnected-(RV108-Pad1)
- RV108 pad 2: Net-(J3-Pin_4) -> Net-(J8-Pin_19)
- RV108 pad 3: Net-(J3-Pin_18) -> Net-(J8-Pin_17)
- RV109 pad 1: unconnected-(RV35-Pad1) -> unconnected-(RV109-Pad1)
- RV109 pad 2: Net-(J4-Pin_4) -> Net-(J9-Pin_2)
- RV109 pad 3: Net-(J4-Pin_20) -> Net-(J9-Pin_4)
- RV110 pad 1: unconnected-(RV36-Pad1) -> unconnected-(RV110-Pad1)
- RV110 pad 2: Net-(J4-Pin_19) -> Net-(J9-Pin_17)
- RV110 pad 3: Net-(J4-Pin_17) -> Net-(J9-Pin_1)
- RV111 pad 1: unconnected-(RV34-Pad1) -> unconnected-(RV111-Pad1)
- RV111 pad 2: Net-(J4-Pin_17) -> Net-(J9-Pin_4)
- RV111 pad 3: Net-(J4-Pin_15) -> Net-(J9-Pin_6)
- RV112 pad 1: unconnected-(RV30-Pad1) -> unconnected-(RV112-Pad1)
- RV112 pad 2: Net-(J4-Pin_4) -> Net-(J9-Pin_4)
- RV112 pad 3: Net-(J4-Pin_16) -> Net-(J9-Pin_8)
- RV113 pad 1: unconnected-(RV27-Pad1) -> unconnected-(RV113-Pad1)
- RV113 pad 2: Net-(J4-Pin_17) -> Net-(J9-Pin_17)
- RV113 pad 3: Net-(J4-Pin_7) -> Net-(J9-Pin_3)
- RV114 pad 1: unconnected-(RV29-Pad1) -> unconnected-(RV114-Pad1)
- RV114 pad 2: Net-(J4-Pin_17) -> Net-(J9-Pin_4)
- RV114 pad 3: Net-(J4-Pin_9) -> Net-(J9-Pin_10)
- RV115 pad 1: unconnected-(RV31-Pad1) -> unconnected-(RV115-Pad1)
- RV115 pad 2: Net-(J4-Pin_17) -> Net-(J9-Pin_17)
- RV115 pad 3: Net-(J4-Pin_11) -> Net-(J9-Pin_5)
- RV116 pad 1: unconnected-(RV33-Pad1) -> unconnected-(RV116-Pad1)
- RV116 pad 2: Net-(J4-Pin_17) -> Net-(J9-Pin_4)
- RV116 pad 3: Net-(J4-Pin_13) -> Net-(J9-Pin_12)
- RV117 pad 1: unconnected-(RV32-Pad1) -> unconnected-(RV117-Pad1)
- RV117 pad 2: Net-(J4-Pin_4) -> Net-(J9-Pin_17)
- RV117 pad 3: Net-(J4-Pin_18) -> Net-(J9-Pin_7)
- RV118 pad 1: unconnected-(RV28-Pad1) -> unconnected-(RV118-Pad1)
- RV118 pad 2: Net-(J4-Pin_4) -> Net-(J9-Pin_4)
- RV118 pad 3: Net-(J4-Pin_14) -> Net-(J9-Pin_14)
- RV119 pad 1: unconnected-(RV26-Pad1) -> unconnected-(RV119-Pad1)
- RV119 pad 2: Net-(J4-Pin_4) -> Net-(J9-Pin_17)
- RV119 pad 3: Net-(J4-Pin_12) -> Net-(J9-Pin_9)
- RV120 pad 1: unconnected-(RV24-Pad1) -> unconnected-(RV120-Pad1)
- RV120 pad 2: Net-(J4-Pin_4) -> Net-(J9-Pin_4)
- RV120 pad 3: Net-(J4-Pin_10) -> Net-(J9-Pin_16)
- RV121 pad 1: unconnected-(RV23-Pad1) -> unconnected-(RV121-Pad1)
- RV121 pad 2: Net-(J4-Pin_17) -> Net-(J9-Pin_17)
- RV121 pad 3: Net-(J4-Pin_3) -> Net-(J9-Pin_11)
- RV122 pad 1: unconnected-(RV25-Pad1) -> unconnected-(RV122-Pad1)
- RV122 pad 2: Net-(J4-Pin_17) -> Net-(J9-Pin_4)
- RV122 pad 3: Net-(J4-Pin_5) -> Net-(J9-Pin_18)
- RV123 pad 1: unconnected-(RV22-Pad1) -> unconnected-(RV123-Pad1)
- RV123 pad 2: Net-(J4-Pin_4) -> Net-(J9-Pin_17)
- RV123 pad 3: Net-(J4-Pin_8) -> Net-(J9-Pin_13)
- RV124 pad 1: unconnected-(RV20-Pad1) -> unconnected-(RV124-Pad1)
- RV124 pad 2: Net-(J4-Pin_17) -> Net-(J9-Pin_17)
- RV124 pad 3: Net-(J4-Pin_1) -> Net-(J9-Pin_15)
- RV125 pad 1: unconnected-(RV21-Pad1) -> unconnected-(RV125-Pad1)
- RV125 pad 2: Net-(J4-Pin_4) -> Net-(J9-Pin_4)
- RV125 pad 3: Net-(J4-Pin_6) -> Net-(J9-Pin_20)
- RV126 pad 1: unconnected-(RV36-Pad1) -> unconnected-(RV126-Pad1)
- RV126 pad 2: Net-(J4-Pin_19) -> Net-(J9-Pin_19)
- RV126 pad 3: Net-(J4-Pin_17) -> Net-(J9-Pin_17)
- RV127 pad 1: unconnected-(RV19-Pad1) -> unconnected-(RV127-Pad1)
- RV127 pad 2: Net-(J4-Pin_2) -> Net-(J10-Pin_2)
- RV127 pad 3: Net-(J4-Pin_4) -> Net-(J10-Pin_4)
- RV128 pad 1: unconnected-(RV17-Pad1) -> unconnected-(RV128-Pad1)
- RV128 pad 2: Net-(J3-Pin_4) -> Net-(J10-Pin_17)
- RV128 pad 3: Net-(J3-Pin_6) -> Net-(J10-Pin_1)
- RV129 pad 1: unconnected-(RV16-Pad1) -> unconnected-(RV129-Pad1)
- RV129 pad 2: Net-(J3-Pin_4) -> Net-(J10-Pin_4)
- RV129 pad 3: Net-(J3-Pin_8) -> Net-(J10-Pin_6)
- RV130 pad 1: unconnected-(RV18-Pad1) -> unconnected-(RV130-Pad1)
- RV130 pad 2: Net-(J3-Pin_2) -> Net-(J10-Pin_4)
- RV130 pad 3: Net-(J3-Pin_4) -> Net-(J10-Pin_8)
- RV131 pad 1: unconnected-(RV12-Pad1) -> unconnected-(RV131-Pad1)
- RV131 pad 2: Net-(J3-Pin_4) -> Net-(J10-Pin_17)
- RV131 pad 3: Net-(J3-Pin_16) -> Net-(J10-Pin_3)
- RV132 pad 1: unconnected-(RV15-Pad1) -> unconnected-(RV132-Pad1)
- RV132 pad 2: Net-(J3-Pin_4) -> Net-(J10-Pin_4)
- RV132 pad 3: Net-(J3-Pin_10) -> Net-(J10-Pin_10)
- RV133 pad 1: unconnected-(RV13-Pad1) -> unconnected-(RV133-Pad1)
- RV133 pad 2: Net-(J3-Pin_4) -> Net-(J10-Pin_17)
- RV133 pad 3: Net-(J3-Pin_14) -> Net-(J10-Pin_5)
- RV134 pad 1: unconnected-(RV14-Pad1) -> unconnected-(RV134-Pad1)
- RV134 pad 2: Net-(J3-Pin_4) -> Net-(J10-Pin_4)
- RV134 pad 3: Net-(J3-Pin_12) -> Net-(J10-Pin_12)
- RV135 pad 1: unconnected-(RV11-Pad1) -> unconnected-(RV135-Pad1)
- RV135 pad 2: Net-(J3-Pin_4) -> Net-(J10-Pin_17)
- RV135 pad 3: Net-(J3-Pin_18) -> Net-(J10-Pin_7)
- RV136 pad 1: unconnected-(RV10-Pad1) -> unconnected-(RV136-Pad1)
- RV136 pad 2: Net-(J3-Pin_4) -> Net-(J10-Pin_4)
- RV136 pad 3: Net-(J3-Pin_20) -> Net-(J10-Pin_14)
- RV137 pad 1: unconnected-(RV31-Pad1) -> unconnected-(RV137-Pad1)
- RV137 pad 2: Net-(J4-Pin_17) -> Net-(J10-Pin_17)
- RV137 pad 3: Net-(J4-Pin_11) -> Net-(J10-Pin_9)
- RV138 pad 1: unconnected-(RV27-Pad1) -> unconnected-(RV138-Pad1)
- RV138 pad 2: Net-(J4-Pin_17) -> Net-(J10-Pin_4)
- RV138 pad 3: Net-(J4-Pin_7) -> Net-(J10-Pin_16)
- RV139 pad 1: unconnected-(RV34-Pad1) -> unconnected-(RV139-Pad1)
- RV139 pad 2: Net-(J4-Pin_17) -> Net-(J10-Pin_17)
- RV139 pad 3: Net-(J4-Pin_15) -> Net-(J10-Pin_11)
- RV140 pad 1: unconnected-(RV29-Pad1) -> unconnected-(RV140-Pad1)
- RV140 pad 2: Net-(J4-Pin_17) -> Net-(J10-Pin_4)
- RV140 pad 3: Net-(J4-Pin_9) -> Net-(J10-Pin_18)
- RV141 pad 1: unconnected-(RV33-Pad1) -> unconnected-(RV141-Pad1)
- RV141 pad 2: Net-(J4-Pin_17) -> Net-(J10-Pin_17)
- RV141 pad 3: Net-(J4-Pin_13) -> Net-(J10-Pin_13)
- RV142 pad 1: unconnected-(RV25-Pad1) -> unconnected-(RV142-Pad1)
- RV142 pad 2: Net-(J4-Pin_17) -> Net-(J10-Pin_17)
- RV142 pad 3: Net-(J4-Pin_5) -> Net-(J10-Pin_15)
- RV143 pad 1: unconnected-(RV20-Pad1) -> unconnected-(RV143-Pad1)
- RV143 pad 2: Net-(J4-Pin_17) -> Net-(J10-Pin_4)
- RV143 pad 3: Net-(J4-Pin_1) -> Net-(J10-Pin_20)
- RV144 pad 1: unconnected-(RV23-Pad1) -> unconnected-(RV144-Pad1)
- RV144 pad 2: Net-(J4-Pin_17) -> Net-(J10-Pin_19)
- RV144 pad 3: Net-(J4-Pin_3) -> Net-(J10-Pin_17)
- RV37 pad 1: unconnected-(RV36-Pad1) -> unconnected-(RV37-Pad1)
- RV37 pad 2: Net-(J4-Pin_19) -> Net-(J5-Pin_2)
- RV37 pad 3: Net-(J4-Pin_17) -> Net-(J5-Pin_4)
- RV38 pad 1: unconnected-(RV35-Pad1) -> unconnected-(RV38-Pad1)
- RV38 pad 2: Net-(J4-Pin_4) -> Net-(J5-Pin_17)
- RV38 pad 3: Net-(J4-Pin_20) -> Net-(J5-Pin_1)
- RV39 pad 1: unconnected-(RV29-Pad1) -> unconnected-(RV39-Pad1)
- RV39 pad 2: Net-(J4-Pin_17) -> Net-(J5-Pin_4)
- RV39 pad 3: Net-(J4-Pin_9) -> Net-(J5-Pin_6)
- RV40 pad 1: unconnected-(RV34-Pad1) -> unconnected-(RV40-Pad1)
- RV40 pad 2: Net-(J4-Pin_17) -> Net-(J5-Pin_4)
- RV40 pad 3: Net-(J4-Pin_15) -> Net-(J5-Pin_8)
- RV41 pad 1: unconnected-(RV33-Pad1) -> unconnected-(RV41-Pad1)
- RV41 pad 2: Net-(J4-Pin_17) -> Net-(J5-Pin_17)
- RV41 pad 3: Net-(J4-Pin_13) -> Net-(J5-Pin_3)
- RV42 pad 1: unconnected-(RV31-Pad1) -> unconnected-(RV42-Pad1)
- RV42 pad 2: Net-(J4-Pin_17) -> Net-(J5-Pin_4)
- RV42 pad 3: Net-(J4-Pin_11) -> Net-(J5-Pin_10)
- RV43 pad 1: unconnected-(RV27-Pad1) -> unconnected-(RV43-Pad1)
- RV43 pad 2: Net-(J4-Pin_17) -> Net-(J5-Pin_17)
- RV43 pad 3: Net-(J4-Pin_7) -> Net-(J5-Pin_5)
- RV44 pad 1: unconnected-(RV30-Pad1) -> unconnected-(RV44-Pad1)
- RV44 pad 2: Net-(J4-Pin_4) -> Net-(J5-Pin_4)
- RV44 pad 3: Net-(J4-Pin_16) -> Net-(J5-Pin_12)
- RV45 pad 1: unconnected-(RV32-Pad1) -> unconnected-(RV45-Pad1)
- RV45 pad 2: Net-(J4-Pin_4) -> Net-(J5-Pin_17)
- RV45 pad 3: Net-(J4-Pin_18) -> Net-(J5-Pin_7)
- RV46 pad 1: unconnected-(RV24-Pad1) -> unconnected-(RV46-Pad1)
- RV46 pad 2: Net-(J4-Pin_4) -> Net-(J5-Pin_4)
- RV46 pad 3: Net-(J4-Pin_10) -> Net-(J5-Pin_14)
- RV47 pad 1: unconnected-(RV26-Pad1) -> unconnected-(RV47-Pad1)
- RV47 pad 2: Net-(J4-Pin_4) -> Net-(J5-Pin_17)
- RV47 pad 3: Net-(J4-Pin_12) -> Net-(J5-Pin_9)
- RV48 pad 1: unconnected-(RV28-Pad1) -> unconnected-(RV48-Pad1)
- RV48 pad 2: Net-(J4-Pin_4) -> Net-(J5-Pin_4)
- RV48 pad 3: Net-(J4-Pin_14) -> Net-(J5-Pin_16)
- RV49 pad 1: unconnected-(RV22-Pad1) -> unconnected-(RV49-Pad1)
- RV49 pad 2: Net-(J4-Pin_4) -> Net-(J5-Pin_17)
- RV49 pad 3: Net-(J4-Pin_8) -> Net-(J5-Pin_11)
- RV50 pad 1: unconnected-(RV23-Pad1) -> unconnected-(RV50-Pad1)
- RV50 pad 2: Net-(J4-Pin_17) -> Net-(J5-Pin_4)
- RV50 pad 3: Net-(J4-Pin_3) -> Net-(J5-Pin_18)
- RV51 pad 1: unconnected-(RV21-Pad1) -> unconnected-(RV51-Pad1)
- RV51 pad 2: Net-(J4-Pin_4) -> Net-(J5-Pin_17)
- RV51 pad 3: Net-(J4-Pin_6) -> Net-(J5-Pin_13)
- RV52 pad 1: unconnected-(RV20-Pad1) -> unconnected-(RV52-Pad1)
- RV52 pad 2: Net-(J4-Pin_17) -> Net-(J5-Pin_17)
- RV52 pad 3: Net-(J4-Pin_1) -> Net-(J5-Pin_15)
- RV53 pad 1: unconnected-(RV19-Pad1) -> unconnected-(RV53-Pad1)
- RV53 pad 2: Net-(J4-Pin_2) -> Net-(J5-Pin_4)
- RV53 pad 3: Net-(J4-Pin_4) -> Net-(J5-Pin_20)
- RV54 pad 1: unconnected-(RV25-Pad1) -> unconnected-(RV54-Pad1)
- RV54 pad 2: Net-(J4-Pin_17) -> Net-(J5-Pin_19)
- RV54 pad 3: Net-(J4-Pin_5) -> Net-(J5-Pin_17)
- RV55 pad 1: unconnected-(RV18-Pad1) -> unconnected-(RV55-Pad1)
- RV55 pad 2: Net-(J3-Pin_2) -> Net-(J6-Pin_2)
- RV55 pad 3: Net-(J3-Pin_4) -> Net-(J6-Pin_4)
- RV56 pad 1: unconnected-(RV16-Pad1) -> unconnected-(RV56-Pad1)
- RV56 pad 2: Net-(J3-Pin_4) -> Net-(J6-Pin_17)
- RV56 pad 3: Net-(J3-Pin_8) -> Net-(J6-Pin_1)
- RV57 pad 1: unconnected-(RV4-Pad1) -> unconnected-(RV57-Pad1)
- RV57 pad 2: Net-(J3-Pin_17) -> Net-(J6-Pin_4)
- RV57 pad 3: Net-(J3-Pin_3) -> Net-(J6-Pin_6)
- RV58 pad 1: unconnected-(RV17-Pad1) -> unconnected-(RV58-Pad1)
- RV58 pad 2: Net-(J3-Pin_4) -> Net-(J6-Pin_4)
- RV58 pad 3: Net-(J3-Pin_6) -> Net-(J6-Pin_8)
- RV59 pad 1: unconnected-(RV6-Pad1) -> unconnected-(RV59-Pad1)
- RV59 pad 2: Net-(J3-Pin_17) -> Net-(J6-Pin_17)
- RV59 pad 3: Net-(J3-Pin_1) -> Net-(J6-Pin_3)
- RV60 pad 1: unconnected-(RV14-Pad1) -> unconnected-(RV60-Pad1)
- RV60 pad 2: Net-(J3-Pin_4) -> Net-(J6-Pin_4)
- RV60 pad 3: Net-(J3-Pin_12) -> Net-(J6-Pin_10)
- RV61 pad 1: unconnected-(RV13-Pad1) -> unconnected-(RV61-Pad1)
- RV61 pad 2: Net-(J3-Pin_4) -> Net-(J6-Pin_17)
- RV61 pad 3: Net-(J3-Pin_14) -> Net-(J6-Pin_5)
- RV62 pad 1: unconnected-(RV5-Pad1) -> unconnected-(RV62-Pad1)
- RV62 pad 2: Net-(J3-Pin_17) -> Net-(J6-Pin_4)
- RV62 pad 3: Net-(J3-Pin_7) -> Net-(J6-Pin_12)
- RV63 pad 1: unconnected-(RV9-Pad1) -> unconnected-(RV63-Pad1)
- RV63 pad 2: Net-(J3-Pin_17) -> Net-(J6-Pin_17)
- RV63 pad 3: Net-(J3-Pin_13) -> Net-(J6-Pin_7)
- RV64 pad 1: unconnected-(RV12-Pad1) -> unconnected-(RV64-Pad1)
- RV64 pad 2: Net-(J3-Pin_4) -> Net-(J6-Pin_4)
- RV64 pad 3: Net-(J3-Pin_16) -> Net-(J6-Pin_14)
- RV65 pad 1: unconnected-(RV8-Pad1) -> unconnected-(RV65-Pad1)
- RV65 pad 2: Net-(J3-Pin_17) -> Net-(J6-Pin_17)
- RV65 pad 3: Net-(J3-Pin_9) -> Net-(J6-Pin_9)
- RV66 pad 1: unconnected-(RV15-Pad1) -> unconnected-(RV66-Pad1)
- RV66 pad 2: Net-(J3-Pin_4) -> Net-(J6-Pin_4)
- RV66 pad 3: Net-(J3-Pin_10) -> Net-(J6-Pin_16)
- RV67 pad 1: unconnected-(RV3-Pad1) -> unconnected-(RV67-Pad1)
- RV67 pad 2: Net-(J3-Pin_17) -> Net-(J6-Pin_17)
- RV67 pad 3: Net-(J3-Pin_11) -> Net-(J6-Pin_11)
- RV68 pad 1: unconnected-(RV7-Pad1) -> unconnected-(RV68-Pad1)
- RV68 pad 2: Net-(J3-Pin_17) -> Net-(J6-Pin_4)
- RV68 pad 3: Net-(J3-Pin_5) -> Net-(J6-Pin_18)
- RV69 pad 1: unconnected-(RV2-Pad1) -> unconnected-(RV69-Pad1)
- RV69 pad 2: Net-(J3-Pin_17) -> Net-(J6-Pin_17)
- RV69 pad 3: Net-(J3-Pin_15) -> Net-(J6-Pin_13)
- RV70 pad 1: unconnected-(RV11-Pad1) -> unconnected-(RV70-Pad1)
- RV70 pad 2: Net-(J3-Pin_4) -> Net-(J6-Pin_17)
- RV70 pad 3: Net-(J3-Pin_18) -> Net-(J6-Pin_15)
- RV71 pad 1: unconnected-(RV10-Pad1) -> unconnected-(RV71-Pad1)
- RV71 pad 2: Net-(J3-Pin_4) -> Net-(J6-Pin_4)
- RV71 pad 3: Net-(J3-Pin_20) -> Net-(J6-Pin_20)
- RV72 pad 1: unconnected-(RV1-Pad1) -> unconnected-(RV72-Pad1)
- RV72 pad 2: Net-(J3-Pin_19) -> Net-(J6-Pin_19)
- RV72 pad 3: Net-(J3-Pin_17) -> Net-(J6-Pin_17)
- RV73 pad 1: unconnected-(RV36-Pad1) -> unconnected-(RV73-Pad1)
- RV73 pad 2: Net-(J4-Pin_19) -> Net-(J7-Pin_2)
- RV73 pad 3: Net-(J4-Pin_17) -> Net-(J7-Pin_4)
- RV74 pad 1: unconnected-(RV35-Pad1) -> unconnected-(RV74-Pad1)
- RV74 pad 2: Net-(J4-Pin_4) -> Net-(J7-Pin_17)
- RV74 pad 3: Net-(J4-Pin_20) -> Net-(J7-Pin_1)
- RV75 pad 1: unconnected-(RV27-Pad1) -> unconnected-(RV75-Pad1)
- RV75 pad 2: Net-(J4-Pin_17) -> Net-(J7-Pin_4)
- RV75 pad 3: Net-(J4-Pin_7) -> Net-(J7-Pin_6)
- RV76 pad 1: unconnected-(RV29-Pad1) -> unconnected-(RV76-Pad1)
- RV76 pad 2: Net-(J4-Pin_17) -> Net-(J7-Pin_4)
- RV76 pad 3: Net-(J4-Pin_9) -> Net-(J7-Pin_8)
- RV77 pad 1: unconnected-(RV28-Pad1) -> unconnected-(RV77-Pad1)
- RV77 pad 2: Net-(J4-Pin_4) -> Net-(J7-Pin_17)
- RV77 pad 3: Net-(J4-Pin_14) -> Net-(J7-Pin_3)
- RV78 pad 1: unconnected-(RV32-Pad1) -> unconnected-(RV78-Pad1)
- RV78 pad 2: Net-(J4-Pin_4) -> Net-(J7-Pin_4)
- RV78 pad 3: Net-(J4-Pin_18) -> Net-(J7-Pin_10)
- RV79 pad 1: unconnected-(RV30-Pad1) -> unconnected-(RV79-Pad1)
- RV79 pad 2: Net-(J4-Pin_4) -> Net-(J7-Pin_17)
- RV79 pad 3: Net-(J4-Pin_16) -> Net-(J7-Pin_5)
- RV80 pad 1: unconnected-(RV26-Pad1) -> unconnected-(RV80-Pad1)
- RV80 pad 2: Net-(J4-Pin_4) -> Net-(J7-Pin_4)
- RV80 pad 3: Net-(J4-Pin_12) -> Net-(J7-Pin_12)
- RV81 pad 1: unconnected-(RV24-Pad1) -> unconnected-(RV81-Pad1)
- RV81 pad 2: Net-(J4-Pin_4) -> Net-(J7-Pin_17)
- RV81 pad 3: Net-(J4-Pin_10) -> Net-(J7-Pin_7)
- RV82 pad 1: unconnected-(RV33-Pad1) -> unconnected-(RV82-Pad1)
- RV82 pad 2: Net-(J4-Pin_17) -> Net-(J7-Pin_4)
- RV82 pad 3: Net-(J4-Pin_13) -> Net-(J7-Pin_14)
- RV83 pad 1: unconnected-(RV31-Pad1) -> unconnected-(RV83-Pad1)
- RV83 pad 2: Net-(J4-Pin_17) -> Net-(J7-Pin_17)
- RV83 pad 3: Net-(J4-Pin_11) -> Net-(J7-Pin_9)
- RV84 pad 1: unconnected-(RV34-Pad1) -> unconnected-(RV84-Pad1)
- RV84 pad 2: Net-(J4-Pin_17) -> Net-(J7-Pin_4)
- RV84 pad 3: Net-(J4-Pin_15) -> Net-(J7-Pin_16)
- RV85 pad 1: unconnected-(RV21-Pad1) -> unconnected-(RV85-Pad1)
- RV85 pad 2: Net-(J4-Pin_4) -> Net-(J7-Pin_17)
- RV85 pad 3: Net-(J4-Pin_6) -> Net-(J7-Pin_11)
- RV86 pad 1: unconnected-(RV20-Pad1) -> unconnected-(RV86-Pad1)
- RV86 pad 2: Net-(J4-Pin_17) -> Net-(J7-Pin_4)
- RV86 pad 3: Net-(J4-Pin_1) -> Net-(J7-Pin_18)
- RV87 pad 1: unconnected-(RV25-Pad1) -> unconnected-(RV87-Pad1)
- RV87 pad 2: Net-(J4-Pin_17) -> Net-(J7-Pin_17)
- RV87 pad 3: Net-(J4-Pin_5) -> Net-(J7-Pin_13)
- RV88 pad 1: unconnected-(RV19-Pad1) -> unconnected-(RV88-Pad1)
- RV88 pad 2: Net-(J4-Pin_2) -> Net-(J7-Pin_17)
- RV88 pad 3: Net-(J4-Pin_4) -> Net-(J7-Pin_15)
- RV89 pad 1: unconnected-(RV23-Pad1) -> unconnected-(RV89-Pad1)
- RV89 pad 2: Net-(J4-Pin_17) -> Net-(J7-Pin_4)
- RV89 pad 3: Net-(J4-Pin_3) -> Net-(J7-Pin_20)
- RV90 pad 1: unconnected-(RV22-Pad1) -> unconnected-(RV90-Pad1)
- RV90 pad 2: Net-(J4-Pin_4) -> Net-(J7-Pin_19)
- RV90 pad 3: Net-(J4-Pin_8) -> Net-(J7-Pin_17)
- RV91 pad 1: unconnected-(RV18-Pad1) -> unconnected-(RV91-Pad1)
- RV91 pad 2: Net-(J3-Pin_2) -> Net-(J8-Pin_2)
- RV91 pad 3: Net-(J3-Pin_4) -> Net-(J8-Pin_4)
- RV92 pad 1: unconnected-(RV4-Pad1) -> unconnected-(RV92-Pad1)
- RV92 pad 2: Net-(J3-Pin_17) -> Net-(J8-Pin_17)
- RV92 pad 3: Net-(J3-Pin_3) -> Net-(J8-Pin_1)
- RV93 pad 1: unconnected-(RV16-Pad1) -> unconnected-(RV93-Pad1)
- RV93 pad 2: Net-(J3-Pin_4) -> Net-(J8-Pin_4)
- RV93 pad 3: Net-(J3-Pin_8) -> Net-(J8-Pin_6)
- RV94 pad 1: unconnected-(RV6-Pad1) -> unconnected-(RV94-Pad1)
- RV94 pad 2: Net-(J3-Pin_17) -> Net-(J8-Pin_4)
- RV94 pad 3: Net-(J3-Pin_1) -> Net-(J8-Pin_8)
- RV95 pad 1: unconnected-(RV17-Pad1) -> unconnected-(RV95-Pad1)
- RV95 pad 2: Net-(J3-Pin_4) -> Net-(J8-Pin_17)
- RV95 pad 3: Net-(J3-Pin_6) -> Net-(J8-Pin_3)
- RV96 pad 1: unconnected-(RV5-Pad1) -> unconnected-(RV96-Pad1)
- RV96 pad 2: Net-(J3-Pin_17) -> Net-(J8-Pin_4)
- RV96 pad 3: Net-(J3-Pin_7) -> Net-(J8-Pin_10)
- RV97 pad 1: unconnected-(RV15-Pad1) -> unconnected-(RV97-Pad1)
- RV97 pad 2: Net-(J3-Pin_4) -> Net-(J8-Pin_17)
- RV97 pad 3: Net-(J3-Pin_10) -> Net-(J8-Pin_5)
- RV98 pad 1: unconnected-(RV8-Pad1) -> unconnected-(RV98-Pad1)
- RV98 pad 2: Net-(J3-Pin_17) -> Net-(J8-Pin_4)
- RV98 pad 3: Net-(J3-Pin_9) -> Net-(J8-Pin_12)
- RV99 pad 1: unconnected-(RV7-Pad1) -> unconnected-(RV99-Pad1)
- RV99 pad 2: Net-(J3-Pin_17) -> Net-(J8-Pin_17)
- RV99 pad 3: Net-(J3-Pin_5) -> Net-(J8-Pin_7)
- U2 pad 1: Net-(J3-Pin_19) -> Net-(J5-Pin_19)
- U2 pad 10: Net-(J4-Pin_17) -> Net-(J6-Pin_17)
- U2 pad 12: Net-(J4-Pin_4) -> Net-(J6-Pin_4)
- U2 pad 14: Net-(J4-Pin_2) -> Net-(J6-Pin_2)
- U2 pad 3: Net-(J3-Pin_17) -> Net-(J5-Pin_17)
- U2 pad 5: Net-(J3-Pin_4) -> Net-(J5-Pin_4)
- U2 pad 7: Net-(J3-Pin_2) -> Net-(J5-Pin_2)
- U2 pad 8: Net-(J4-Pin_19) -> Net-(J6-Pin_19)
- U3 pad 1: Net-(J3-Pin_19) -> Net-(J7-Pin_19)
- U3 pad 10: Net-(J4-Pin_17) -> Net-(J8-Pin_17)
- U3 pad 12: Net-(J4-Pin_4) -> Net-(J8-Pin_4)
- U3 pad 14: Net-(J4-Pin_2) -> Net-(J8-Pin_2)
- U3 pad 3: Net-(J3-Pin_17) -> Net-(J7-Pin_17)
- U3 pad 5: Net-(J3-Pin_4) -> Net-(J7-Pin_4)
- U3 pad 7: Net-(J3-Pin_2) -> Net-(J7-Pin_2)
- U3 pad 8: Net-(J4-Pin_19) -> Net-(J8-Pin_19)
- U4 pad 1: Net-(J3-Pin_19) -> Net-(J9-Pin_19)
- U4 pad 10: Net-(J4-Pin_17) -> Net-(J10-Pin_17)
- U4 pad 12: Net-(J4-Pin_4) -> Net-(J10-Pin_4)
- U4 pad 14: Net-(J4-Pin_2) -> Net-(J10-Pin_2)
- U4 pad 3: Net-(J3-Pin_17) -> Net-(J9-Pin_17)
- U4 pad 5: Net-(J3-Pin_4) -> Net-(J9-Pin_4)
- U4 pad 7: Net-(J3-Pin_2) -> Net-(J9-Pin_2)
- U4 pad 8: Net-(J4-Pin_19) -> Net-(J10-Pin_19)
Routing:
- removed copper zone on B.Cu, net GND
- removed copper zone on F.Cu, net GND
Other:
- board outline removed
